Commit message: udpate

File: ur_description/urdf/common.gazebo.xacro (robot description, xacro)
@@ -1,4 +1,7 @@
 <?xml version="1.0"?>
-<robot xmlns:xacro="http://ros.org/wiki/xacro">
+<robot xmlns:xacro="http://ros.org/wiki/xacro"
+       xmlns:sensor="http://playerstage.sourceforge.net/gazebo/xmlschema/#sensor"
+       xmlns:controller="http://playerstage.sourceforge.net/gazebo/xmlschema/#controller"
+       xmlns:interface="http://playerstage.sourceforge.net/gazebo/xmlschema/#interface">
   <gazebo>
     <plugin name="ros_control" filename="libgazebo_ros_control.so">
@@ -21,3 +24,80 @@
 -->
   </gazebo>
+  <gazebo reference="link_feed1">
+    <selfCollide>true</selfCollide>
+    <mu1>0.5</mu1>
+    <mu2>0.5</mu2>
+    <kd>1</kd>
+    <kp>7000</kp>
+  </gazebo>
+  <gazebo reference="link_feed2">
+    <selfCollide>true</selfCollide>
+    <mu1>0.5</mu1>
+    <mu2>0.5</mu2>
+    <kd>1</kd>
+    <kp>7000</kp>
+  </gazebo>
+  <gazebo reference="base_link">
+    <selfCollide>true</selfCollide>
+    <mu1>0.5</mu1>
+    <mu2>0.5</mu2>
+    <kd>1</kd>
+    <kp>7000</kp>
+  </gazebo>
+  <gazebo reference="shoulder_link">
+    <selfCollide>true</selfCollide>
+  </gazebo>
+  <gazebo reference="upper_arm_link">
+    <selfCollide>true</selfCollide>
+  </gazebo>
+  <gazebo reference="forearm_link">
+    <selfCollide>true</selfCollide>
+  </gazebo>
+  <gazebo reference="wrist_1_link">
+    <selfCollide>true</selfCollide>
+  </gazebo>
+  <gazebo reference="wrist_2_link">
+    <selfCollide>true</selfCollide>
+  </gazebo>
+  <gazebo reference="wrist_3_link">
+    <selfCollide>true</selfCollide>
+    <mu1>0.5</mu1>
+    <mu2>0.5</mu2>
+    <kd>1</kd>
+    <kp>7000</kp>
+  </gazebo>
+  <gazebo reference="ee_link">
+    <selfCollide>true</selfCollide>
+    <mu1>0.5</mu1>
+    <mu2>0.5</mu2>
+    <kd>1</kd>
+    <kp>7000</kp>
+  </gazebo>
+  <gazebo reference="forcesensor_link">
+    <selfCollide>true</selfCollide>
+    <mu1>0.5</mu1>
+    <mu2>0.5</mu2>
+    <kd>1</kd>
+    <kp>7000</kp>
+    <sensor name="forcesensor_link_contact_sensor" type="contact">
+      <always_on>1</always_on>
+      <update_rate>1000</update_rate>
+      <contact>
+        <collision>forcesensor_link_collision</collision>
+        <topic>/contact_forces</topic>
+      </contact>
+      <plugin name="forcesensor_link_bumper" filename="libreload_contact_sensor_plugin.so">
+        <robotNamespace>/</robotNamespace>
+        <bumperTopicName>/impedance_controller/contact_forces</bumperTopicName>
+        <frameName>forcesensor_link</frameName>
+      </plugin>
+    </sensor>
+  </gazebo>
+  <gazebo reference="bolt_link">
+    <selfCollide>true</selfCollide>
+    <mu1>0.5</mu1>
+    <mu2>0.5</mu2>
+    <kd>1</kd>
+    <kp>7000</kp>
+  </gazebo>
 </robot>

File: ur_description/urdf/ur10.urdf.xacro (robot description, xacro)
@@ -78,8 +78,37 @@
       </xacro:cylinder_inertial>
     </link>
+    <joint name="pedistal_joint" type="fixed">
+      <parent link="${prefix}base_link" />
+      <child link = "${prefix}pedistal_link" />
+      <origin xyz="0.0 0.0 0.0" rpy="0.0 0.0 0.0" />
+    </joint>
+    <link name="${prefix}pedistal_link">
+      <visual>
+        <geometry>
+          <box size="0.15 0.15 0.90" />
+        </geometry>
+        <material name="LightGrey">
+          <color rgba="0.7 0.7 0.7 1.0"/>
+        </material>
+        <origin xyz="0 0 0.45" rpy="0 0 0" />
+      </visual>
+      <collision>
+        <geometry>
+          <box size="0.15 0.15 0.90" />
+        </geometry>
+        <origin xyz="0 0 0.45" rpy="0 0 0" />
+      </collision>
+      <inertial>
+        <mass value="1" />
+        <origin xyz="0 0 0.45" rpy="0 0 0" />
+        <inertia ixx="1.0" ixy="0.0" ixz="0.0"
+                           iyy="0.0" iyz="0.0"
+                                     izz="1.0" />
+      </inertial>
+    </link>
     <joint name="${prefix}shoulder_pan_joint" type="revolute">
-      <parent link="${prefix}base_link" />
+      <parent link="${prefix}pedistal_link" />
       <child link = "${prefix}shoulder_link" />
-      <origin xyz="0.0 0.0 ${shoulder_height}" rpy="0.0 0.0 0.0" />
+      <origin xyz="0.0 0.0 ${shoulder_height+0.9}" rpy="0.0 0.0 0.0" />
       <axis xyz="0 0 1" />
       <xacro:unless value="${joint_limited}">
@@ -112,5 +141,5 @@
       <parent link="${prefix}shoulder_link" />
       <child link = "${prefix}upper_arm_link" />
-      <origin xyz="0.0 ${shoulder_offset} 0.0" rpy="0.0 ${pi / 2.0} 0.0" />
+      <origin xyz="0.0 ${shoulder_offset} 0.0" rpy="0.0 ${pi / 2.0 * 0.5} 0.0" />
       <axis xyz="0 1 0" />
       <xacro:unless value="${joint_limited}">
@@ -143,5 +172,5 @@
       <parent link="${prefix}upper_arm_link" />
       <child link = "${prefix}forearm_link" />
-      <origin xyz="0.0 ${elbow_offset} ${upper_arm_length}" rpy="0.0 0.0 0.0" />
+      <origin xyz="0.0 ${elbow_offset} ${upper_arm_length}" rpy="0.0 ${pi / 2.0 * 0.5} 0.0" />
       <axis xyz="0 1 0" />
       <xacro:unless value="${joint_limited}">
@@ -276,4 +305,54 @@
         <origin rpy="0 0 0" xyz="-0.01 0 0"/>
       </collision>
+    </link>
+    <joint name="${prefix}forcesensor_fixed_joint" type="fixed">
+      <parent link="${prefix}ee_link" />
+      <child link = "${prefix}forcesensor_link" />
+      <origin xyz="0.0175 0.0 0.0" rpy="0.0 ${pi/2} 0.0" />
+    </joint>
+    <link name="${prefix}forcesensor_link">
+      <visual>
+        <geometry>
+          <cylinder radius="0.035" length="0.035" />
+        </geometry>
+        <material name="LightGrey">
+          <color rgba="0.7 0.7 0.7 1.0"/>
+        </material>
+        <origin rpy="0 0 0" xyz="0 0 0.0"/>
+      </visual>
+      <collision>
+        <geometry>
+          <cylinder radius="0.0175" length="0.07" />
+        </geometry>
+        <origin rpy="0 0 0" xyz="0 0 0.0"/>
+      </collision>
+      <xacro:cylinder_inertial radius="0.0175" length="0.07" mass="0.200">
+        <origin xyz="0.0 0.0 0.0" rpy="0 0 0" />
+      </xacro:cylinder_inertial>
+    </link>
+    <joint name="${prefix}bolt_fixed_joint" type="fixed">
+      <parent link="${prefix}forcesensor_link" />
+      <child link = "${prefix}bolt_link" />
+      <origin xyz="0 0 ${0.0075+0.0175}" rpy="0.0 0.0 0.0" />
+    </joint>
+    <link name="${prefix}bolt_link">
+      <visual>
+        <geometry>
+          <cylinder radius="0.0075" length="2.0" />
+        </geometry>
+        <material name="LightGrey">
+          <color rgba="0.7 0.7 0.7 1.0"/>
+        </material>
+        <origin rpy="0 ${pi/2} 0" xyz="0 0 0"/>
+      </visual>
+      <collision>
+        <geometry>
+          <cylinder radius="0.0075" length="2.0" />
+        </geometry>
+        <origin rpy="0 ${pi/2} 0" xyz="0 0 0"/>
+      </collision>
+      <xacro:cylinder_inertial radius="0.0075" length="2.0" mass="0.200">
+        <origin xyz="0.0 0.0 0.0" rpy="0 ${pi/2} 0" />
+      </xacro:cylinder_inertial>
     </link>
     <xacro:ur_arm_transmission prefix="${prefix}" hardware_interface="${hardware_interface}" />

Commit message: udpate

File: ur_description/urdf/common.gazebo.xacro (robot description, xacro)
@@ -24,4 +24,10 @@
 -->
   </gazebo>
+  <gazebo reference="world">
+    <selfCollide>true</selfCollide>
+  </gazebo>
+  <gazebo reference="base_link">
+    <selfCollide>true</selfCollide>
+  </gazebo>
   <gazebo reference="link_feed1">
     <selfCollide>true</selfCollide>
@@ -38,25 +44,21 @@
     <kp>7000</kp>
   </gazebo>
-  <gazebo reference="base_link">
-    <selfCollide>true</selfCollide>
-    <mu1>0.5</mu1>
-    <mu2>0.5</mu2>
-    <kd>1</kd>
-    <kp>7000</kp>
+  <gazebo reference="ur10_base_link">
+    <selfCollide>false</selfCollide>
   </gazebo>
   <gazebo reference="shoulder_link">
-    <selfCollide>true</selfCollide>
+    <selfCollide>false</selfCollide>
   </gazebo>
   <gazebo reference="upper_arm_link">
-    <selfCollide>true</selfCollide>
+    <selfCollide>false</selfCollide>
   </gazebo>
   <gazebo reference="forearm_link">
-    <selfCollide>true</selfCollide>
+    <selfCollide>false</selfCollide>
   </gazebo>
   <gazebo reference="wrist_1_link">
-    <selfCollide>true</selfCollide>
+    <selfCollide>false</selfCollide>
   </gazebo>
   <gazebo reference="wrist_2_link">
-    <selfCollide>true</selfCollide>
+    <selfCollide>false</selfCollide>
   </gazebo>
   <gazebo reference="wrist_3_link">

File: ur_description/urdf/feed.urdf.xacro (robot description, xacro)
@@ -1,4 +1,11 @@
 <?xml version="1.0"?>
-<robot xmlns:xacro="http://ros.org/wiki/xacro">
+<robot name="feeds" xmlns:xacro="http://ros.org/wiki/xacro">
+  <link name="world" />
+  <link name="base_link" />
+  <joint name="world_base_joint" type="fixed">
+    <parent link="world"/>
+    <child link="base_link"/>
+    <origin xyz="0 0 0" rpy="0 0 0"/>
+  </joint>
   <link name="link_feed1">
     <visual>
@@ -26,5 +33,5 @@
   </link>
   <joint name="joint_feed1_to_base_link" type="fixed">
-    <parent link="world"/>
+    <parent link="base_link"/>
     <child link="link_feed1"/>
     <origin xyz="-1.25 1.5 0" rpy="1.57079632679 0 0"/>
@@ -57,5 +64,5 @@
     <parent link="world"/>
     <child link="link_feed2"/>
-    <origin xyz="3.2 0.075 0" rpy="1.57079632679 -1.57079632679 0"/>
+    <origin xyz="1.2 0.075 0" rpy="1.57079632679 -1.57079632679 0"/>
   </joint>
 </robot>

File: ur_description/urdf/ur10.urdf.xacro (robot description, xacro)
@@ -60,27 +60,4 @@
 		 wrist_2_lower_limit:=${-pi}    wrist_2_upper_limit:=${pi}
 		 wrist_3_lower_limit:=${-pi}    wrist_3_upper_limit:=${pi}">
-    <link name="${prefix}base_link" >
-      <visual>
-        <geometry>
-          <mesh filename="package://ur_description/meshes/ur10/visual/base.dae"/>
-        </geometry>
-        <material name="LightGrey">
-          <color rgba="0.7 0.7 0.7 1.0"/>
-        </material>
-      </visual>
-      <collision>
-        <geometry>
-          <mesh filename="package://ur_description/meshes/ur10/collision/base.stl"/>
-        </geometry>
-      </collision>
-      <xacro:cylinder_inertial radius="0.075" length="0.038" mass="${base_mass}">
-        <origin xyz="0.0 0.0 0.0" rpy="0 0 0" />
-      </xacro:cylinder_inertial>
-    </link>
-    <joint name="pedistal_joint" type="fixed">
-      <parent link="${prefix}base_link" />
-      <child link = "${prefix}pedistal_link" />
-      <origin xyz="0.0 0.0 0.0" rpy="0.0 0.0 0.0" />
-    </joint>
     <link name="${prefix}pedistal_link">
       <visual>
@@ -91,5 +68,5 @@
           <color rgba="0.7 0.7 0.7 1.0"/>
         </material>
-        <origin xyz="0 0 0.45" rpy="0 0 0" />
+        <origin xyz="0 0 0.0" rpy="0 0 0" />
       </visual>
       <collision>
@@ -97,18 +74,41 @@
           <box size="0.15 0.15 0.90" />
         </geometry>
-        <origin xyz="0 0 0.45" rpy="0 0 0" />
+        <origin xyz="0 0 0.0" rpy="0 0 0" />
       </collision>
       <inertial>
         <mass value="1" />
-        <origin xyz="0 0 0.45" rpy="0 0 0" />
+        <origin xyz="0 0 0.0" rpy="0 0 0" />
         <inertia ixx="1.0" ixy="0.0" ixz="0.0"
-                           iyy="0.0" iyz="0.0"
+                           iyy="1.0" iyz="0.0"
                                      izz="1.0" />
       </inertial>
     </link>
+    <joint name="pedistal_joint" type="fixed">
+      <parent link="${prefix}pedistal_link" />
+      <child link = "${prefix}ur10_base_link" />
+      <origin xyz="0.0 0.0 ${0.45}" rpy="0.0 0.0 0.0" />
+    </joint>
+    <link name="${prefix}ur10_base_link" >
+      <visual>
+        <geometry>
+          <mesh filename="package://ur_description/meshes/ur10/visual/base.dae"/>
+        </geometry>
+        <material name="LightGrey">
+          <color rgba="0.7 0.7 0.7 1.0"/>
+        </material>
+      </visual>
+      <collision>
+        <geometry>
+          <mesh filename="package://ur_description/meshes/ur10/collision/base.stl"/>
+        </geometry>
+      </collision>
+      <xacro:cylinder_inertial radius="0.075" length="0.038" mass="${base_mass}">
+        <origin xyz="0.0 0.0 0.0" rpy="0 0 0" />
+      </xacro:cylinder_inertial>
+    </link>
     <joint name="${prefix}shoulder_pan_joint" type="revolute">
-      <parent link="${prefix}pedistal_link" />
+      <parent link="${prefix}ur10_base_link" />
       <child link = "${prefix}shoulder_link" />
-      <origin xyz="0.0 0.0 ${shoulder_height+0.9}" rpy="0.0 0.0 0.0" />
+      <origin xyz="0.0 0.0 ${shoulder_height}" rpy="0.0 0.0 0.0" />
       <axis xyz="0 0 1" />
       <xacro:unless value="${joint_limited}">

File: ur_description/urdf/ur10_robot.urdf.xacro (robot description, xacro)
@@ -8,6 +8,7 @@
   <!-- arm -->
   <xacro:ur10_robot prefix="" joint_limited="false" hardware_interface="EffortJointInterface" />
-  <xacro:include filename="$(find ur_description)/urdf/feed.urdf.xacro" />
+  <!--xacro:include filename="$(find ur_description)/urdf/feed.urdf.xacro" /-->
   <link name="world" />
+  <link name="base_link" />
   <joint name="world_joint" type="fixed">
     <parent link="world" />
@@ -15,3 +16,8 @@
     <origin xyz="0.0 0.0 0.0" rpy="0.0 0.0 0.0" />
   </joint>
+  <joint name="base_joint" type="fixed">
+    <parent link="base_link" />
+    <child link = "pedistal_link" />
+    <origin xyz="0.0 0.0 0.45" rpy="0.0 0.0 0.0" />
+  </joint>
 </robot>

File: ur_description/urdf/ur10_robot_generated.urdf (robot description, URDF)
Before this commit: robot ur10, 16 links, 15 joints
Links:
- removed link link_feed1
- removed link link_feed2
- added link ur10_base_link, mass 4.0; collision mesh filename=package://ur_description/meshes/ur10/collision/base.stl; visual mesh filename=package://ur_description/meshes/ur10/visual/base.dae
- link base_link: mass 4.0 -> None; geometry 
Joints:
- removed joint joint_feed1_to_base_link
- removed joint joint_feed2_to_base_link
- added joint base_joint: type fixed, parent base_link, child pedistal_link, origin xyz=0.0 0.0 0.45 rpy=0.0 0.0 0.0
- joint pedistal_joint: child pedistal_link -> ur10_base_link; origin xyz=0.0 0.0 0.0 rpy=0.0 0.0 0.0 -> xyz=0.0 0.0 0.45 rpy=0.0 0.0 0.0; parent base_link -> pedistal_link
- joint shoulder_pan_joint: origin xyz=0.0 0.0 1.0273 rpy=0.0 0.0 0.0 -> xyz=0.0 0.0 0.1273 rpy=0.0 0.0 0.0; parent pedistal_link -> ur10_base_link

Commit message: reverting to cannonical and adding namespace

File: ur_description/urdf/common.gazebo.xacro (robot description, xacro)
@@ -6,5 +6,5 @@
   <gazebo>
     <plugin name="ros_control" filename="libgazebo_ros_control.so">
-      <!--robotNamespace>/</robotNamespace-->
+      <robotNamespace>/amici</robotNamespace>
       <!--robotSimType>gazebo_ros_control/DefaultRobotHWSim</robotSimType-->
     </plugin>

File: ur_description/urdf/ur10.urdf.xacro (robot description, xacro)
@@ -60,34 +60,5 @@
 		 wrist_2_lower_limit:=${-pi}    wrist_2_upper_limit:=${pi}
 		 wrist_3_lower_limit:=${-pi}    wrist_3_upper_limit:=${pi}">
-    <link name="${prefix}pedistal_link">
-      <visual>
-        <geometry>
-          <box size="0.15 0.15 0.90" />
-        </geometry>
-        <material name="LightGrey">
-          <color rgba="0.7 0.7 0.7 1.0"/>
-        </material>
-        <origin xyz="0 0 0.0" rpy="0 0 0" />
-      </visual>
-      <collision>
-        <geometry>
-          <box size="0.15 0.15 0.90" />
-        </geometry>
-        <origin xyz="0 0 0.0" rpy="0 0 0" />
-      </collision>
-      <inertial>
-        <mass value="1" />
-        <origin xyz="0 0 0.0" rpy="0 0 0" />
-        <inertia ixx="1.0" ixy="0.0" ixz="0.0"
-                           iyy="1.0" iyz="0.0"
-                                     izz="1.0" />
-      </inertial>
-    </link>
-    <joint name="pedistal_joint" type="fixed">
-      <parent link="${prefix}pedistal_link" />
-      <child link = "${prefix}ur10_base_link" />
-      <origin xyz="0.0 0.0 ${0.45}" rpy="0.0 0.0 0.0" />
-    </joint>
-    <link name="${prefix}ur10_base_link" >
+    <link name="${prefix}base_link" >
       <visual>
         <geometry>
@@ -108,5 +79,5 @@
     </link>
     <joint name="${prefix}shoulder_pan_joint" type="revolute">
-      <parent link="${prefix}ur10_base_link" />
+      <parent link="${prefix}base_link" />
       <child link = "${prefix}shoulder_link" />
       <origin xyz="0.0 0.0 ${shoulder_height}" rpy="0.0 0.0 0.0" />
@@ -141,5 +112,5 @@
       <parent link="${prefix}shoulder_link" />
       <child link = "${prefix}upper_arm_link" />
-      <origin xyz="0.0 ${shoulder_offset} 0.0" rpy="0.0 ${pi / 2.0 * 0.5} 0.0" />
+      <origin xyz="0.0 ${shoulder_offset} 0.0" rpy="0.0 ${pi / 2.0} 0.0" />
       <axis xyz="0 1 0" />
       <xacro:unless value="${joint_limited}">
@@ -172,5 +143,5 @@
       <parent link="${prefix}upper_arm_link" />
       <child link = "${prefix}forearm_link" />
-      <origin xyz="0.0 ${elbow_offset} ${upper_arm_length}" rpy="0.0 ${pi / 2.0 * 0.5} 0.0" />
+      <origin xyz="0.0 ${elbow_offset} ${upper_arm_length}" rpy="0.0 0.0 0.0" />
       <axis xyz="0 1 0" />
       <xacro:unless value="${joint_limited}">
@@ -305,54 +276,4 @@
         <origin rpy="0 0 0" xyz="-0.01 0 0"/>
       </collision>
-    </link>
-    <joint name="${prefix}forcesensor_fixed_joint" type="fixed">
-      <parent link="${prefix}ee_link" />
-      <child link = "${prefix}forcesensor_link" />
-      <origin xyz="0.0175 0.0 0.0" rpy="0.0 ${pi/2} 0.0" />
-    </joint>
-    <link name="${prefix}forcesensor_link">
-      <visual>
-        <geometry>
-          <cylinder radius="0.035" length="0.035" />
-        </geometry>
-        <material name="LightGrey">
-          <color rgba="0.7 0.7 0.7 1.0"/>
-        </material>
-        <origin rpy="0 0 0" xyz="0 0 0.0"/>
-      </visual>
-      <collision>
-        <geometry>
-          <cylinder radius="0.0175" length="0.07" />
-        </geometry>
-        <origin rpy="0 0 0" xyz="0 0 0.0"/>
-      </collision>
-      <xacro:cylinder_inertial radius="0.0175" length="0.07" mass="0.200">
-        <origin xyz="0.0 0.0 0.0" rpy="0 0 0" />
-      </xacro:cylinder_inertial>
-    </link>
-    <joint name="${prefix}bolt_fixed_joint" type="fixed">
-      <parent link="${prefix}forcesensor_link" />
-      <child link = "${prefix}bolt_link" />
-      <origin xyz="0 0 ${0.0075+0.0175}" rpy="0.0 0.0 0.0" />
-    </joint>
-    <link name="${prefix}bolt_link">
-      <visual>
-        <geometry>
-          <cylinder radius="0.0075" length="2.0" />
-        </geometry>
-        <material name="LightGrey">
-          <color rgba="0.7 0.7 0.7 1.0"/>
-        </material>
-        <origin rpy="0 ${pi/2} 0" xyz="0 0 0"/>
-      </visual>
-      <collision>
-        <geometry>
-          <cylinder radius="0.0075" length="2.0" />
-        </geometry>
-        <origin rpy="0 ${pi/2} 0" xyz="0 0 0"/>
-      </collision>
-      <xacro:cylinder_inertial radius="0.0075" length="2.0" mass="0.200">
-        <origin xyz="0.0 0.0 0.0" rpy="0 ${pi/2} 0" />
-      </xacro:cylinder_inertial>
     </link>
     <xacro:ur_arm_transmission prefix="${prefix}" hardware_interface="${hardware_interface}" />

File: ur_description/urdf/ur10_robot.urdf.xacro (robot description, xacro)
@@ -7,5 +7,5 @@
   <xacro:include filename="$(find ur_description)/urdf/ur10.urdf.xacro" />
   <!-- arm -->
-  <xacro:ur10_robot prefix="" joint_limited="false" hardware_interface="EffortJointInterface" />
+  <xacro:ur10_robot prefix="" joint_limited="false" hardware_interface="VelocityJointInterface" />
   <!--xacro:include filename="$(find ur_description)/urdf/feed.urdf.xacro" /-->
   <link name="world" />
